File: speedo.sch (KiCad schematic (older format))
At the start: 51 parts, among them J1 Conn_01x08, J2 Conn_01x10, J3 Prog Header, Q1 BSS138, SW1 SW_Push, U1 US1881, U2 LT1762-3.3, U3 4N25, U4 LT1762-5, U5 ATMEGA644-20AU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

Commit message: Finished first layout of pcb
Parts:
- removed C21, C22: 100nF, Capacitors_SMD:C_0603, symbol C
- removed U6: ADuM1200BR, Housings_SOIC:SOIC-8_3.9x4.9mm_Pitch1.27mm, symbol ADuM1200BR
- added D4, D5: D, Diodes_SMD:D_SOD-123F, symbol D
- added R13: 18K, Resistors_SMD:R_0603, symbol R
- J1: footprint Connectors_Molex:Molex_PicoBlade_53047-0810_08x1.25mm_Straight -> Connectors_Molex:Molex_PicoBlade_53398-0871_08x1.25mm_Straight
- J2: footprint Connectors_Molex:Molex_PicoBlade_53047-1010_10x1.25mm_Straight -> Connectors_Molex:Molex_PicoBlade_53398-1071_10x1.25mm_Straight
- U2, U4: footprint Housings_SSOP:MSOP-8-1EP_3x3mm_Pitch0.65mm -> Housings_SSOP:MSOP-8_3x3mm_Pitch0.65mm
- U5: footprint Housings_QFP:TQFP-44-1EP_10x10mm_Pitch0.8mm -> Housings_QFP:TQFP-44_10x10mm_Pitch0.8mm
- Y1: value 10MHz 18pF -> 16MHz 18pF
Connections:
- net GPIO1 is gone; now on net LM35-POS: J2.7 (Pin_7)
- net GPIO2 is gone; now on net LM35-NEG: J2.8 (Pin_8)
- net +3V3: no longer J3.6 (Pin_6)
- net BUTTON1: now also U5.40 ((PCINT8/T0/XCK)PB0); no longer U5.24 ((PCINT21/TDI)PC5)
- net BUTTON2: now also U5.42 ((PCINT10/AIN0/INT2)PB2); no longer U5.25 ((PCINT22/TOSC1)PC6)
- net GND: now also D4.1 (K), R13.2
- net HALL-EFF: now also U5.11 ((PCINT26/INT0)PD2); no longer U5.40 ((PCINT8/T0/XCK)PB0)
- net LCD-CS: now also U5.44 ((PCINT12/OC0B/~SS~)PB4); no longer U5.13 ((PCINT28/OC1B)PD4)
- net LCD-DC: now also U5.13 ((PCINT28/OC1B)PD4); no longer U5.22 ((PCINT19/TMS)PC3)
- net LCD-LED: now also U5.14 ((PCINT294/OC1A)PD5); no longer U5.16 ((PCINT31/OC2A)PD7)
- net LCD-RST: now also U5.12 ((PCINT27/INT1)PD3); no longer U5.21 ((PCINT18/TCK)PC2)
- net RX: now also J2.9 (Pin_9); no longer J2.10 (Pin_10)
- net TX: now also J2.10 (Pin_10); no longer J2.9 (Pin_9)
- net LM35-POS: now reaches U5.34 ((PCINT3/ADC3)PA3)
- net LM35-POS: now also R13.1
- net LM35-NEG: now reaches U5.35 ((PCINT2/ADC2)PA2)
- net LM35-NEG: now also D5.2 (A)
- net GPIO1-ISO: no longer names the net of U5.30 ((PCINT7/ADC7)PA7)
- net GPIO2-ISO: no longer names the net of U5.31 ((PCINT6/ADC6)PA6)
- new net: D4.2 (A), D5.1 (K)
- no-connect marks 1 -> 2
Other:
- note added: "LM35-POS is the signal pin\nLM35-NEG is the ground pin\nThe power pin on LM35 connected to 5V"
- moved on the sheet: R9
