File: speedo.kicad_pcb (KiCad board)
At the start: 4 copper layers, 70 x 34 mm, 53 parts, among them J1 Conn_01x08, J2 Conn_01x10, J3 Prog Header, Q1 BSS138, SW1 SW_Push, U1 US1881, U2 LT1762-3.3, U3 4N25, U4 LT1762-5, U5 ATMEGA644-20AU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

Commit message: Fixed solder mask clearance
Other:
- rule pad_to_mask_clearance: 0.2 -> 0.0381
Changed lines of the file:
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@@
     (pad_size 1.524 1.524)
     (pad_drill 0.762)
-    (pad_to_mask_clearance 0.2)
+    (pad_to_mask_clearance 0.0381)
     (aux_axis_origin 0 0)
     (visible_elements FFFEFF7F)
